Commit message: IFARLAB Environment

File: ifarlab_description/urdf/ifarlab_description.urdf (robot description, URDF)
Before this commit: robot ifarlab, 15 links, 14 joints
Links:
- added link sick_camera, mass 0.8666400000000004; collision mesh filename=file:////home/cem/colcon_ws/src/ifarlab/ifarlab_description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 scale=0.001 0.001 0.001; visual mesh filename=file:////home/cem/colcon_ws/src/ifarlab/ifarlab_description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 scale=0.001 0.001 0.001
- link tool0: mass 0.3126115786693621 -> 0.22117646672670696
Joints:
- added joint tool0-sick_joint: type fixed, parent tool0, child sick_camera, origin xyz=0.050329 0.003 -0.017406 rpy=0 0 0
- joint flange-tool0: origin xyz=0 0.031 0 rpy=0 0 0 -> xyz=0 0.032 -0.02 rpy=0 0 0
- joint wrist_3-flange: origin xyz=0 0 0.0423 rpy=1.5707963267948966 0 0 -> xyz=0 0 0.0 rpy=1.5707963267948966 0 0

Commit message: Last version

File: ifarlab_description/urdf/ifarlab_description.urdf (robot description, URDF)
Before this commit: robot ifarlab, 16 links, 15 joints
Links:
- removed link chassis
Joints:
- removed joint chassis_joint

File: ifarlab_description/urdf/ur10e_transmissions.xacro (robot description, xacro)
@@ -56,4 +56,13 @@
       </actuator>
     </transmission>
+    <transmission name="${prefix}linear_axis_trans">
+      <type>transmission_interface/SimpleTransmission</type>
+      <joint name="linear_axis_moving_joint">
+        <hardwareInterface>${hw_interface}</hardwareInterface>
+      </joint>
+      <actuator name="${prefix}linear_axis_motor">
+        <mechanicalReduction>1</mechanicalReduction>
+      </actuator>
+    </transmission>
   </xacro:macro>
 </robot>
